File: tinynode.kicad_sch (KiCad schematic)
At the start: 6 parts, among them J1 Conn_01x04, J2 Conn_Coaxial, J3 Conn_01x04, J4 Conn_01x04, U1 SHT31-DIS

Commit message: Initial commit (stm32 v1)
Parts:
- removed BT1: Battery_Cell, symbol Device:Battery_Cell
- removed U1: SHT31-DIS, Sensor_Humidity:Sensirion_DFN-8-1EP_2.5x2.5mm_P0.5mm_EP1.1x1.7mm, symbol Sensor_Humidity:SHT31-DIS
- added C1, C6, C8, C9: 10u, Capacitor_SMD:C_0603_1608Metric, symbol Device:C_Small
- added C10: 0.1u, Capacitor_SMD:C_0603_1608Metric, symbol Device:C_Small
- added C2: 10u, Capacitor_SMD:CP_Elec_4x5.4, symbol Device:C_Polarized_Small
- added C3: 220nF, Capacitor_SMD:C_0603_1608Metric, symbol Device:C_Small
- added C4, C5, C7: 100n, Capacitor_SMD:C_0603_1608Metric, symbol Device:C_Small
- added D2: D_Schottky_Small, Diode_SMD:D_SOD-123, symbol Device:D_Schottky_Small
- added D3: D_Schottky, Diode_SMD:D_SOD-123, symbol Device:D_Schottky
- added H1, H2, H3, H4: MountingHole_Pad, MountingHole:MountingHole_3.2mm_M3_Pad_Via, symbol Mechanical:MountingHole_Pad
- added J1: Conn_01x04, stary:BK-18650-PC4, symbol Connector_Generic:Conn_01x04
- added J2: USB_C_Receptacle_USB2.0_16P, Connector_USB:USB_C_Receptacle_HRO_TYPE-C-31-M-12, symbol Connector:USB_C_Receptacle_USB2.0_16P
- added J7: Conn_01x08, Connector_JST:JST_SH_SM08B-SRSS-TB_1x08-1MP_P1.00mm_Horizontal, symbol Connector_Generic:Conn_01x08
- added J8: Conn_01x02, Connector_JST:JST_XH_B2B-XH-A_1x02_P2.50mm_Vertical, symbol Connector_Generic:Conn_01x02
- added J9: Conn_01x02, Connector_JST:JST_PH_B2B-PH-K_1x02_P2.00mm_Vertical, symbol Connector_Generic:Conn_01x02
- added L1: 2.2u, Inductor_SMD:L_1008_2520Metric, symbol Device:L_Small
- added L2: SRP7050WA-101M, Inductor_SMD:L_Bourns_SRP7028A_7.3x6.6mm, symbol Device:L_Small
- added Q1, Q2, Q3: AO3401A, Package_TO_SOT_SMD:SOT-23, symbol Transistor_FET:AO3401A
- added Q4: 2N7002K, Package_TO_SOT_SMD:SOT-23, symbol Transistor_FET:2N7002K
- added R1, R19: 100k, Resistor_SMD:R_0603_1608Metric, symbol Device:R_Small
- added R10: 56k, Resistor_SMD:R_0603_1608Metric, symbol Device:R_Small
- added R11: 1.18k, Resistor_SMD:R_0603_1608Metric, symbol Device:R_Small
- added R12: 50m, Resistor_SMD:R_1210_3225Metric, symbol Device:R_Small
- added R13, R7, R8: R_Small, Resistor_SMD:R_0603_1608Metric, symbol Device:R_Small
- added R14: 1m, Resistor_SMD:R_0603_1608Metric, symbol Device:R_Small
- added R15: 500k, Resistor_SMD:R_0603_1608Metric, symbol Device:R_Small
- added R16, R17, R18: 0.1, Resistor_SMD:R_1206_3216Metric, symbol Device:R_Small
- added R2: 120, Resistor_SMD:R_0603_1608Metric, symbol Device:R_Small
- added R20: 100, Resistor_SMD:R_0603_1608Metric, symbol Device:R_Small
- added R21, R5, R6: 0, Resistor_SMD:R_0402_1005Metric, symbol Device:R_Small
- added R3, R4: 5.1k, Resistor_SMD:R_0603_1608Metric, symbol Device:R_Small
- added R9: 178k, Resistor_SMD:R_0603_1608Metric, symbol Device:R_Small
- added SW1: SW_Push, Button_Switch_SMD:SW_Tactile_SPST_NO_Straight_CK_PTS636Sx25SMTRLFS, symbol Switch:SW_Push
- added U1: APX803L40-33SA-7, Package_TO_SOT_SMD:SOT-23-3, symbol stary:APX803L
- added U2: TLV62568DDC, Package_TO_SOT_SMD:SOT-23-6, symbol Regulator_Switching:TLV62568DDC
- added U3: CN3791, Package_SO:SSOP-10_3.9x4.9mm_P1.00mm, symbol stary:CN3791
- added U4: CH340N, Package_SO:SOP-8_3.9x4.9mm_P1.27mm, symbol Interface_USB:CH340N
- added U5: CN3163, Package_SO:SOIC-8-1EP_3.9x4.9mm_P1.27mm_EP2.41x3.3mm_ThermalVias, symbol stary:CN3163
- added U6: LoRa-E5, wio:LoRa-E5, symbol wio:LoRa-E5
- added U7: INA3221, Package_DFN_QFN:Texas_RGV0016A_VQFN-16-1EP_4x4mm_P0.65mm_EP2.1x2.1mm, symbol Power_Management:INA3221
- added U8: XB3306D, Package_TO_SOT_SMD:SOT-23-3, symbol stary:XB3306D
- J3: renamed from J2; footprint (none) -> Connector_Coaxial:SMA_Amphenol_901-144_Vertical
- J4: renamed from J1; footprint (none) -> Connector_PinHeader_2.54mm:PinHeader_1x04_P2.54mm_Vertical
- J5: renamed from J3; footprint (none) -> Connector_PinHeader_2.54mm:PinHeader_1x04_P2.54mm_Vertical
- J6: renamed from J4; footprint (none) -> Connector_PinHeader_2.54mm:PinHeader_1x04_P2.54mm_Vertical
Connections:
- net +3V3: now also J5.1 (Pin_1), J6.1 (Pin_1), J7.7 (Pin_7), R18.2, U4.5 (VCC), U4.8 (V3), U6.1 (VCC), U7.1 (IN-3)
- net GND: now also J5.4 (Pin_4), J6.4 (Pin_4), C1.2, C2.2, C3.2, C5.2, C6.2, C7.2, C8.2, C9.2, D2.2 (A), H1.1, H2.1, H3.1, H4.1, J2.A1 (GND), J2.A12 (GND), J2.B1 (GND), J2.B12 (GND), J2.S1 (SHIELD), J7.1 (Pin_1), J8.1 (Pin_1), Q4.2 (S), R10.2, R11.2, R13.1, R15.2, R3.2, R4.2, R8.2, SW1.2, U1.1 (GND), U2.2 (GND), U3.2 (GND), U4.3 (GND), U5.1 (TEMP), U5.3 (GND), U5.9 (EPAD), U6.14 (GND), U6.16 (GND), U6.2 (GND), U6.22 (GND), U7.17 (EP), U7.3 (GND), U8.1 (VM)
- net sda: now reaches J5.2 (Pin_2)
- net sda: now also R21.2, U6.5 (PB15), U7.7 (SDA)
- net scl: now reaches J5.3 (Pin_3)
- net scl: now also U6.6 (PA15), U7.6 (SCL)
- net at J3.1 (In): now also U6.15 (RFIO)
- net lpuart1_tx: now reaches J4.2 (Pin_2)
- net lpuart1_tx: now also U6.13 (PC0)
- net lpuart1_rx: now reaches J4.3 (Pin_3)
- net lpuart1_rx: now also U6.12 (PC1)
- net uart2_tx: now reaches J6.2 (Pin_2)
- net uart2_tx: now also J7.3 (Pin_3), U6.19 (PA2)
- net uart2_rx: now reaches J6.3 (Pin_3)
- net uart2_rx: now also J7.6 (Pin_6), U6.18 (PA3)
- new net: J2.B8 (SBU2), R6.2
- new net: R1.2, U1.2 (~{RESET}), U2.1 (EN)
- new net: R11.1, U5.2 (ISET)
- new net: L2.2, R12.1, U3.8 (CSP)
- new net: R2.1, U3.5 (COM)
- new net: C3.1, R2.2
- new net: C4.2, U3.1 (VG)
- new net: Q1.1 (G), U3.10 (DRV)
- new net: R10.1, R9.2, U3.6 (MPPT)
- new net: Q3.1 (G), Q4.3 (D), R19.2
- new net: J7.8 (Pin_8), Q3.3 (D)
- new net: C10.1, R20.1, U8.2 (VDD)
- new net: R21.1, U7.5 (A0)
- new net: J2.B5 (CC2), R4.1
- new net: L1.1, U2.3 (SW)
- new net: R7.2, R8.1, U2.6 (FB)
- new net: J2.A8 (SBU1), R5.1
- new net: J2.A5 (CC1), R3.1
- new net: SW1.1, U6.17 (RST)
- new net !charging: U5.7 (~{CHRG})
- new net !done: U5.6 (~{DONE})
- new net +5V: D3.2 (A), J2.A4 (VBUS), J2.A9 (VBUS), J2.B4 (VBUS), J2.B9 (VBUS), Q2.1 (G), R13.2, U5.4 (VIN)
- new net 3v3_pre: C7.1, C8.1, L1.2, R18.1, R7.1, U7.16 (VPU), U7.2 (IN+3), U7.4 (VS)
- new net Vin: C9.1, D3.1 (K), Q2.3 (D), Q3.2 (S), R1.1, R19.1, U1.3 (VCC), U2.4 (VIN)
- new net batt+_ina: C6.1, Q2.2 (S), R12.2, R16.2, U3.7 (BAT), U5.5 (BAT), U5.8 (FB), U7.11 (IN-1)
- new net batt+_pre: J1.1 (Pin_1), J1.2 (Pin_2), J9.1 (Pin_1), R14.1, R16.1, R20.2, U7.12 (IN+1)
- new net batt-_unprot: C10.2, J1.3 (Pin_3), J1.4 (Pin_4), J9.2 (Pin_2), U8.3 (GND)
- new net batt_adc: R14.2, R15.1
- new net lte_en: U6.11 (PB5)
- new net lte_netlight: J7.5 (Pin_5)
- new net lte_pwrkey: J7.2 (Pin_2), U6.21 (PA9)
- new net lte_reset: J7.4 (Pin_4), U6.20 (PB10)
- new net solar_in: J8.2 (Pin_2), R17.1, U7.15 (IN+2)
- new net solar_in_ina: C1.1, C2.1, C4.1, C5.1, Q1.2 (S), R17.2, R9.1, U3.9 (VCC), U7.14 (IN-2)
- new net solar_sw: D2.1 (K), L2.1, Q1.3 (D)
- new net spi2_cs: U6.25 (PB9)
- new net spi2_miso: U6.26 (PB14)
- new net spi2_mosi: U6.27 (PA10)
- new net spi2_sck: U6.24 (PB13~{})
- new net swclk: R6.1, U6.4 (PA14)
- new net swdio: R5.2, U6.3 (PA13)
- new net uart1_rx: U4.6 (TXD), U6.9 (PB7)
- new net uart1_tx: U4.7 (RXD), U6.10 (PB6)
- new net usb_d+: J2.A6 (D+), J2.B6 (D+), U4.1 (UD+)
- new net usb_d-: J2.A7 (D-), J2.B7 (D-), U4.2 (UD-)
- new net ~{lte_en}: Q4.1 (G)
- no-connect marks 0 -> 11
Other:
- note added: "1A charge current"
- note added: "For Meshtastic, use address 0x42 (SDA connected to A0)"
- note added: "LTE????"
- note added: "Power supply to +, Load to -"
- note added: "Solar in"
- note added: "Wurth 865080340001"
- note added: "load sharing for charging circuit"
- note removed: "Battery charger. How do?"
- note removed: "MPPT - myself?"
- note removed: "cn3791"
- moved on the sheet: J3, J4, J5, J6
