File: hardware/stm32-v1/tinynode.kicad_pcb (KiCad board)
At the start: 4 copper layers, 80 x 60 mm, 61 parts, among them J1 Conn_01x04, J2 USB_C_Receptacle_USB2.0_16P, J3 Conn_Coaxial, J4 Conn_01x04, J5 Conn_01x04, J6 Conn_01x04, J7 Conn_01x08, J8 Conn_01x02, J9 Conn_01x02, Q1 AO3401A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

Commit message: v1 as fabbed
Parts:
- added C11: 100n, Capacitor_SMD:C_0603_1608Metric, F.Cu at (181.8, 117.1)
- added C12: 100n, Capacitor_SMD:C_0603_1608Metric, F.Cu at (182.6, 86.9)
- added C13: 100n, Capacitor_SMD:C_0603_1608Metric, F.Cu at (183.0, 94.5)
- added R22: 5.1k, Resistor_SMD:R_0603_1608Metric, F.Cu at (173.7, 98.0)
- added R23: 5.1k, Resistor_SMD:R_0603_1608Metric, F.Cu at (175.3, 98.0)
- added U9: AHT20, stary:AHT20, F.Cu at (181.9, 113.3)
- L2: value SRP7050WA-101M -> SRP7050WA-100M
- R13: value R_Small -> 100k
- R7: value R_Small -> 115k
- R8: value R_Small -> 25.5k
- moved R15 56.8 mm to (180.0, 101.7)
- moved R14 56.8 mm to (180.0, 100.2)
Connections:
- U6 pad 7: unconnected-(U6-PB4-Pad7) -> /batt_adc
Routing:
- net +3V3: track 196.7 -> 252.7 mm, vias 7 -> 8
- net /sda: track 89.2 -> 132.9 mm, vias 4 -> 5
- net /scl: track 84.5 -> 121.4 mm, vias 2 -> 3
- net /batt_adc: track 1.50 -> 8.81 mm
- net GND: track 62.8 -> 69.1 mm, vias 31 -> 34
- net /batt+_pre: track 130.7 -> 134.2 mm, vias 1 -> 2
- net /solar_in_ina: track 63.0 -> 61.8 mm
Other:
- outline, holes or cut-outs redrawn
- board text added: "AHT20 Temp+RH"
- board text added: "Smol Meshtastic STM32 node Chloe 2025"
- board text added: "USB-Serial"
