File: hardware/stm32-v1/tinynode.kicad_sch (KiCad schematic)
At the start: 61 parts, among them J1 Conn_01x04, J2 USB_C_Receptacle_USB2.0_16P, J3 Conn_Coaxial, J4 Conn_01x04, J5 Conn_01x04, J6 Conn_01x04, J7 Conn_01x08, J8 Conn_01x02, J9 Conn_01x02, Q1 AO3401A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

Commit message: v1 as fabbed
Parts:
- added C11, C12, C13: 100n, Capacitor_SMD:C_0603_1608Metric, symbol Device:C_Small
- added R22, R23: 5.1k, Resistor_SMD:R_0603_1608Metric, symbol Device:R_Small
- added U9: AHT20, stary:AHT20, symbol stary:AHT20
- L2: value SRP7050WA-101M -> SRP7050WA-100M
- R13: value R_Small -> 100k
- R7: value R_Small -> 115k
- R8: value R_Small -> 25.5k
Connections:
- net +3V3: now also C11.1, C12.1, C13.1, R22.1, R23.1, U9.2 (VDD)
- net GND: now also C11.2, C12.2, C13.2, U9.5 (GND)
- net batt_adc: now also U6.7 (PB4)
- net scl: now also R23.2, U9.3 (SCL)
- net sda: now also R22.2, U9.4 (SDA)
- no-connect marks 11 -> 10
Other:
- note added: "Use JLC04161H-7628, 50ohm on L1 with L2 reference = 0.3493mm thickness"
- moved on the sheet: J3, SW1, U6
